Commit message: them giao dien va huong dan su dung web UI

File: src/kuka_kr3_support/urdf/kr3r540.urdf (robot description, URDF)
Before this commit: robot kuka_kr3r540, 10 links, 9 joints
Links:
- link base_link: geometry collision mesh filename=package://kuka_kr3_support/meshes/kr3r540/collision/base_li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; visual mesh filename=package://kuka_kr3_support/meshes/kr3r540/visual/base_link.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
- link link_1: geometry collision mesh filename=package://kuka_kr3_support/meshes/kr3r540/collision/link_1.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; visual mesh filename=package://kuka_kr3_support/meshes/kr3r540/visual/link_1.stl
- link link_2: geometry collision mesh filename=package://kuka_kr3_support/meshes/kr3r540/collision/link_2.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; visual mesh filename=package://kuka_kr3_support/meshes/kr3r540/visual/link_2.stl
- link link_3: geometry collision mesh filename=package://kuka_kr3_support/meshes/kr3r540/collision/link_3.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; visual mesh filename=package://kuka_kr3_support/meshes/kr3r540/visual/link_3.stl
- link link_4: geometry collision mesh filename=package://kuka_kr3_support/meshes/kr3r540/collision/link_4.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; visual mesh filename=package://kuka_kr3_support/meshes/kr3r540/visual/link_4.stl
- link link_5: geometry collision mesh filename=package://kuka_kr3_support/meshes/kr3r540/collision/link_5.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; visual mesh filename=package://kuka_kr3_support/meshes/kr3r540/visual/link_5.stl
- link link_6: geometry collision mesh filename=package://kuka_kr3_support/meshes/kr3r540/collision/link_6.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; visual mesh filename=package://kuka_kr3_support/meshes/kr3r540/visual/link_6.stl
